Commit message: Refactor URDF

File: workspaceRos/src/phantomx/phantomx_description/urdf/phantomx.xacro (robot description, xacro)
@@ -1,14 +1,14 @@
 <?xml version="1.0" ?>
 <robot name="PhantomX"  xmlns:xacro="http://www.ros.org/wiki/xacro">
-  <xacro:include filename="$(find phantomx_description)/urdf/phantomx_urdf.xacro" />
-  <link name="base_link"/>
-  <xacro:phantomx parent="base_link">
-      <origin xyz="0 0 0" rpy="0 0 0" />
-  </xacro:phantomx>
-  <gazebo>
-    <plugin filename="libgazebo_ros_control.so" name="gazebo_ros_control">
-      <robotNamespace>/phantomx</robotNamespace>
-      <legacyModeNS>true</legacyModeNS>
-    </plugin>
-  </gazebo>
+    <xacro:include filename="$(find phantomx_description)/urdf/phantomx_urdf.xacro" />
+    <link name="base_link"/>
+    <xacro:phantomx parent="base_link">
+        <origin xyz="0 0 0" rpy="0 0 0" />
+    </xacro:phantomx>
+    <gazebo>
+        <plugin filename="libgazebo_ros_control.so" name="gazebo_ros_control">
+            <robotNamespace>/phantomx</robotNamespace>
+            <legacyModeNS>true</legacyModeNS>
+        </plugin>
+    </gazebo>
 </robot>

File: workspaceRos/src/phantomx/phantomx_description/urdf/phantomx_urdf.xacro (robot description, xacro)
@@ -1,243 +1,229 @@
 <?xml version="1.0" ?>
 <robot xmlns:xacro="http://www.ros.org/wiki/xacro">
-<xacro:property name="connect_offset" value="0.02633" />
-<xacro:property name="thigh_offset_y" value="-0.0645" />
-<xacro:property name="thigh_offset_z" value="-0.0145" />
-<xacro:macro name="phantomx" params="parent *origin">
-      <joint name="j_phantomx_attachment" type="fixed">
-        <parent link="${parent}"/>
-        <child link="MP_BODY"/>
-        <insert_block name="origin" />
-      </joint>
-<!--      <gazebo reference="j_phantomx_attachment">-->
-<!--        <implicitSpringDamper>1</implicitSpringDamper>-->
-<!--      </gazebo>-->
-      <link name="MP_BODY">
-        <inertial>
-          <origin xyz="0 0 0" />
-          <mass value="0.97559947"/>
-          <inertia ixx="3.1081800"  ixy="-0.25460189"  ixz="2.0318174" iyy="6.3787776" iyz="0.16417863" izz="5.3316425" />
-        </inertial>
-        <visual>
-          <!--origin xyz="-0.0235 0 -0.03525" rpy="0 0 0" /-->
-          <origin xyz="0 0 0" rpy="0 0 0" />
-          <geometry>
-            <!--box size="0.102 0.109 0.106" /-->
-            <mesh filename="package://phantomx_description/meshes/body.STL"  scale="1 1 1"/>
-          </geometry>
-          <material name="Grey">
-            <color rgba="0.20 0.20 0.20 1.0"/>
-          </material>
-        </visual>
-        <collision>
-          <origin xyz="0 0 0" rpy="0 0 0" />
-          <geometry>
-            <mesh filename="package://phantomx_description/meshes/body_coll.STL"  scale="1 1 1"/>
-          </geometry>
-        </collision>
-      </link>
-      <gazebo reference="MP_BODY">
-        <material>Gazebo/Grey</material>
-      </gazebo>
-    <xacro:leg_l xyz="0.1248 -0.06164  0.001116"  rpy="0 4.7123 0.7853981633974483" suffix="rf"/>
-    <xacro:leg_l xyz="0 -0.1034  0.001116"  rpy="0 4.7123 0" suffix="rm"/>
-    <xacro:leg_l xyz="-0.1248 -0.06164  0.001116"  rpy="0 4.7123 -0.7853981633974483" suffix="rr"/>
-    <xacro:leg_l xyz="0.1248 0.06164  0.001116"  rpy="0 4.7123 2.356194490192345" suffix="lf"/>
-    <xacro:leg_l xyz="0 0.1034  0.001116"  rpy="0 4.7123 3.14159" suffix="lm"/>
-    <xacro:leg_l xyz="-0.1248 0.06164  0.001116"  rpy="0 4.7123 3.9269908169872414" suffix="lr"/>
-</xacro:macro>
- <xacro:macro name="leg_l" params="xyz rpy suffix">
-  <link name="c1_${suffix}">
-    <inertial>
-      <origin xyz="0 -${connect_offset} 0" rpy="0 0 0"  />
-      <mass value="0.324357719"/>
-     <inertia ixx="0.0051411124"  ixy="-0.00057530255"  ixz="-0.000024729049" iyy="0.0081915737" iyz="-0.000019223094" izz="0.0011379812" />
-    </inertial>
-    <visual>
-      <origin xyz="0 -0.0252 0" rpy="0 0 0"  />
-      <geometry>
-        <!--box size="0.045 0.022 0.0325" /-->
-        <mesh filename="package://phantomx_description/meshes/connect.STL"  scale="1 1 1"/>
-      </geometry>
-      <material name="Grey">
-        <color rgba="0.20 0.20 0.20 1.0"/>
-      </material>
-    </visual>
-    <collision>
-      <origin xyz="0 -${connect_offset} 0" rpy="0 0 0"  />
-      <geometry>
-        <mesh filename="package://phantomx_description/meshes/connect_coll.STL"  scale="1 1 1"/>
-      </geometry>
-    </collision>
-  </link>
-  <gazebo reference="c1_${suffix}">
-      <dampingFactor>0.0005</dampingFactor>
-  </gazebo>
-  <link name="c2_${suffix}">
-    <inertial>
-      <origin xyz="0 -${connect_offset} 0" rpy="0 0 0"  />
-      <mass value="0.324357719"/>
-     <inertia ixx="0.0051411124"  ixy="-0.00057530255"  ixz="-0.000024729049" iyy="0.0081915737" iyz="-0.000019223094" izz="0.0011379812" />
-    </inertial>
-    <visual>
-      <origin xyz="0 -0.0252 0" rpy="0 0 0"  />
-      <geometry>
-        <!--box size="0.045 0.022 0.0325" /-->
-        <mesh filename="package://phantomx_description/meshes/connect.STL"  scale="1 1 1"/>
-      </geometry>
-      <material name="Grey">
-        <color rgba="0.20 0.20 0.20 1.0"/>
-      </material>
-    </visual>
-    <collision>
-      <origin xyz="0 -${connect_offset} 0" rpy="0 0 0"  />
-      <geometry>
-        <mesh filename="package://phantomx_description/meshes/connect_coll.STL"  scale="1 1 1"/>
-      </geometry>
-    </collision>
-  </link>
-  <gazebo reference="c2_${suffix}">
-      <dampingFactor>0.0005</dampingFactor>
-  </gazebo>
-  <link name="thigh_${suffix}">
-    <inertial>
-      <origin xyz="0 0 0" rpy="0 0 0"  />
-      <mass value="0.324357719"/>
-     <inertia ixx="0.0051411124"  ixy="-0.00057530255"  ixz="-0.000024729049" iyy="0.0081915737" iyz="-0.000019223094" izz="0.0011379812" />
-    </inertial>
-    <visual>
-      <origin xyz="0 0 0" rpy="0 0 0"  />
-      <geometry>
-        <!--box size="0.045 0.022 0.0325" /-->
-        <mesh filename="package://phantomx_description/meshes/thigh_l.STL"  scale="1 1 1"/>
-      </geometry>
-      <material name="Grey">
-        <color rgba="0.20 0.20 0.20 1.0"/>
-      </material>
-    </visual>
-    <collision>
-      <origin xyz="0 0 0" rpy="0 0 0"  />
-      <geometry>
-        <mesh filename="package://phantomx_description/meshes/thigh_l_coll.STL"  scale="1 1 1"/>
-      </geometry>
-    </collision>
-  </link>
-  <gazebo reference="thigh_${suffix}">
-      <dampingFactor>0.0005</dampingFactor>
-  </gazebo>
-  <link name="tibia_${suffix}">
-    <inertial>
-      <origin xyz="0 0 0" rpy="0 0 0"  />
-      <mass value="0.324357719"/>
-     <inertia ixx="0.0051411124"  ixy="-0.00057530255"  ixz="-0.000024729049" iyy="0.0081915737" iyz="-0.000019223094" izz="0.0011379812" />
-    </inertial>
-    <visual>
-      <origin xyz="0 0 0" rpy="0 0 0"  />
-      <geometry>
-        <!--box size="0.045 0.022 0.0325" /-->
-        <mesh filename="package://phantomx_description/meshes/tibia_l.STL"  scale="1 1 1"/>
-      </geometry>
-      <material name="Grey">
-        <color rgba="0.20 0.20 0.20 1.0"/>
-      </material>
-    </visual>
-    <collision>
-      <origin xyz="0 0 0" rpy="0 0 0"  />
-      <geometry>
-        <mesh filename="package://phantomx_description/meshes/tibia_l_coll.STL"  scale="1 1 1"/>
-      </geometry>
-    </collision>
-  </link>
-    <gazebo reference="tibia_${suffix}">
-        <mu1>50.0</mu1>
-        <mu2>50.0</mu2>
-        <fdir1>0.000000 0.000000 0.000000</fdir1>
-        <kp>500000.0</kp>
-        <kd>10.0</kd>
-        <maxVel>0.00</maxVel>
-        <minDepth>0.001</minDepth>
-        <dampingFactor>0.0005</dampingFactor>
-        <selfCollide>1</selfCollide>
-    </gazebo>
-<!--    <gazebo reference="j_c1_${suffix}">-->
-<!--        <implicitSpringDamper>1</implicitSpringDamper>-->
-<!--    </gazebo>-->
-<!--    <gazebo reference="j_c2_${suffix}">-->
-<!--        <implicitSpringDamper>1</implicitSpringDamper>-->
-<!--    </gazebo>-->
-  <joint name="j_c1_${suffix}" type="revolute">
-    <parent link="MP_BODY"/>
-    <child link="c1_${suffix}"/>
-    <origin xyz="${xyz}" rpy="${rpy}" />
-    <axis xyz="1 0 0" />
-    <limit effort="2.8" velocity="5.6548668" lower="-2.6179939" upper="2.6179939" />
-  </joint>
-  <joint name="j_c2_${suffix}" type="fixed">
-    <parent link="c1_${suffix}"/>
-    <child link="c2_${suffix}"/>
-    <origin xyz="0 -0.054 0" rpy="0 1.5704 3.14159" />
-  </joint>
-  <joint name="j_thigh_${suffix}" type="revolute">
-    <parent link="c2_${suffix}"/>
-    <child link="thigh_${suffix}"/>
-    <origin xyz="0 0 0" rpy=" 0 3.14159 3.14159" />
-    <axis xyz="1 0 0" />
-    <limit effort="2.8" velocity="5.6548668" lower="-2.6179939" upper="2.6179939" />
-  </joint>
-  <joint name="j_tibia_${suffix}" type="revolute">
-    <parent link="thigh_${suffix}"/>
-    <child link="tibia_${suffix}"/>
-    <origin xyz="0 ${thigh_offset_y} ${thigh_offset_z}" rpy="-1.5707 0 3.14159" />
-    <axis xyz="1 0 0" />
-    <limit effort="2.8" velocity="5.6548668" lower="-2.6179939" upper="2.6179939" />
-  </joint>
-<!--  <gazebo reference="j_thigh_${suffix}">-->
-<!--    <implicitSpringDamper>1</implicitSpringDamper>-->
-<!--  </gazebo>-->
-<!--  <gazebo reference="j_tibia_${suffix}">-->
-<!--    <implicitSpringDamper>1</implicitSpringDamper>-->
-<!--  </gazebo>-->
-   <transmission name="t_c1_${suffix}">
-    <type>transmission_interface/SimpleTransmission</type>
-    <joint name="j_c1_${suffix}">
-      <hardwareInterface>hardware_interface/EffortJointInterface</hardwareInterface>
-    </joint>
-    <actuator name="m_c1_${suffix}">
-      <hardwareInterface>hardware_interface/EffortJointInterface</hardwareInterface>
-      <mechanicalReduction>1</mechanicalReduction>
-    </actuator>
-  </transmission>
-   <transmission name="t_thigh_${suffix}">
-    <type>transmission_interface/SimpleTransmission</type>
-    <joint name="j_thigh_${suffix}">
-      <hardwareInterface>hardware_interface/EffortJointInterface</hardwareInterface>
-    </joint>
-    <actuator name="m_thigh_${suffix}">
-      <hardwareInterface>hardware_interface/EffortJointInterface</hardwareInterface>
-      <mechanicalReduction>1</mechanicalReduction>
-    </actuator>
-  </transmission>
-   <transmission name="t_tibia_${suffix}">
-    <type>transmission_interface/SimpleTransmission</type>
-    <joint name="j_tibia_${suffix}">
-      <hardwareInterface>hardware_interface/EffortJointInterface</hardwareInterface>
-    </joint>
-    <actuator name="m_tibia_${suffix}">
-      <hardwareInterface>hardware_interface/EffortJointInterface</hardwareInterface>
-      <mechanicalReduction>1</mechanicalReduction>
-    </actuator>
-  </transmission>
-  <gazebo reference="c1_${suffix}">
-    <material>Gazebo/Grey</material>
-  </gazebo>
-  <gazebo reference="c2_${suffix}">
-    <material>Gazebo/Grey</material>
-  </gazebo>
-  <gazebo reference="thigh_${suffix}">
-    <material>Gazebo/Grey</material>
-  </gazebo>
-  <gazebo reference="tibia_${suffix}">
-    <material>Gazebo/Grey</material>
-  </gazebo>
-</xacro:macro>
+    <xacro:property name="connect_offset" value="0.02633"/>
+    <xacro:property name="thigh_offset_y" value="-0.0645"/>
+    <xacro:property name="thigh_offset_z" value="-0.0145"/>
+    <xacro:macro name="phantomx" params="parent *origin">
+        <joint name="j_phantomx_attachment" type="fixed">
+            <parent link="${parent}"/>
+            <child link="MP_BODY"/>
+            <insert_block name="origin"/>
+        </joint>
+        <link name="MP_BODY">
+            <inertial>
+                <origin xyz="0 0 0"/>
+                <mass value="0.97559947"/>
+                <inertia ixx="3.1081800" ixy="-0.25460189" ixz="2.0318174" iyy="6.3787776" iyz="0.16417863"
+                         izz="5.3316425"/>
+            </inertial>
+            <visual>
+                <origin xyz="0 0 0" rpy="0 0 0"/>
+                <geometry>
+                    <mesh filename="package://phantomx_description/meshes/body.STL" scale="1 1 1"/>
+                </geometry>
+                <material name="Grey">
+                    <color rgba="0.20 0.20 0.20 1.0"/>
+                </material>
+            </visual>
+            <collision>
+                <origin xyz="0 0 0" rpy="0 0 0"/>
+                <geometry>
+                    <mesh filename="package://phantomx_description/meshes/body_coll.STL" scale="1 1 1"/>
+                </geometry>
+            </collision>
+        </link>
+        <gazebo reference="MP_BODY">
+            <material>Gazebo/Grey</material>
+        </gazebo>
+        <xacro:leg_l xyz="0.1248 -0.06164  0.001116" rpy="0 4.7123 0.7853981633974483" suffix="rf"/>
+        <xacro:leg_l xyz="0 -0.1034  0.001116" rpy="0 4.7123 0" suffix="rm"/>
+        <xacro:leg_l xyz="-0.1248 -0.06164  0.001116" rpy="0 4.7123 -0.7853981633974483" suffix="rr"/>
+        <xacro:leg_l xyz="0.1248 0.06164  0.001116" rpy="0 4.7123 2.356194490192345" suffix="lf"/>
+        <xacro:leg_l xyz="0 0.1034  0.001116" rpy="0 4.7123 3.14159" suffix="lm"/>
+        <xacro:leg_l xyz="-0.1248 0.06164  0.001116" rpy="0 4.7123 3.9269908169872414" suffix="lr"/>
+    </xacro:macro>
+    <xacro:macro name="leg_l" params="xyz rpy suffix">
+        <link name="c1_${suffix}">
+            <inertial>
+                <origin xyz="0 -${connect_offset} 0" rpy="0 0 0"/>
+                <mass value="0.324357719"/>
+                <inertia ixx="0.0051411124" ixy="-0.00057530255" ixz="-0.000024729049" iyy="0.0081915737"
+                         iyz="-0.000019223094" izz="0.0011379812"/>
+            </inertial>
+            <visual>
+                <origin xyz="0 -0.0252 0" rpy="0 0 0"/>
+                <geometry>
+                    <!--box size="0.045 0.022 0.0325" /-->
+                    <mesh filename="package://phantomx_description/meshes/connect.STL" scale="1 1 1"/>
+                </geometry>
+                <material name="Grey">
+                    <color rgba="0.20 0.20 0.20 1.0"/>
+                </material>
+            </visual>
+            <collision>
+                <origin xyz="0 -${connect_offset} 0" rpy="0 0 0"/>
+                <geometry>
+                    <mesh filename="package://phantomx_description/meshes/connect_coll.STL" scale="1 1 1"/>
+                </geometry>
+            </collision>
+        </link>
+        <gazebo reference="c1_${suffix}">
+            <dampingFactor>0.0005</dampingFactor>
+        </gazebo>
+        <link name="c2_${suffix}">
+            <inertial>
+                <origin xyz="0 -${connect_offset} 0" rpy="0 0 0"/>
+                <mass value="0.324357719"/>
+                <inertia ixx="0.0051411124" ixy="-0.00057530255" ixz="-0.000024729049" iyy="0.0081915737"
+                         iyz="-0.000019223094" izz="0.0011379812"/>
+            </inertial>
+            <visual>
+                <origin xyz="0 -0.0252 0" rpy="0 0 0"/>
+                <geometry>
+                    <!--box size="0.045 0.022 0.0325" /-->
+                    <mesh filename="package://phantomx_description/meshes/connect.STL" scale="1 1 1"/>
+                </geometry>
+                <material name="Grey">
+                    <color rgba="0.20 0.20 0.20 1.0"/>
+                </material>
+            </visual>
+            <collision>
+                <origin xyz="0 -${connect_offset} 0" rpy="0 0 0"/>
+                <geometry>
+                    <mesh filename="package://phantomx_description/meshes/connect_coll.STL" scale="1 1 1"/>
+                </geometry>
+            </collision>
+        </link>
+        <gazebo reference="c2_${suffix}">
+            <dampingFactor>0.0005</dampingFactor>
+        </gazebo>
+        <link name="thigh_${suffix}">
+            <inertial>
+                <origin xyz="0 0 0" rpy="0 0 0"/>
+                <mass value="0.324357719"/>
+                <inertia ixx="0.0051411124" ixy="-0.00057530255" ixz="-0.000024729049" iyy="0.0081915737"
+                         iyz="-0.000019223094" izz="0.0011379812"/>
+            </inertial>
+            <visual>
+                <origin xyz="0 0 0" rpy="0 0 0"/>
+                <geometry>
+                    <mesh filename="package://phantomx_description/meshes/thigh_l.STL" scale="1 1 1"/>
+                </geometry>
+                <material name="Grey">
+                    <color rgba="0.20 0.20 0.20 1.0"/>
+                </material>
+            </visual>
+            <collision>
+                <origin xyz="0 0 0" rpy="0 0 0"/>
+                <geometry>
+                    <mesh filename="package://phantomx_description/meshes/thigh_l_coll.STL" scale="1 1 1"/>
+                </geometry>
+            </collision>
+        </link>
+        <gazebo reference="thigh_${suffix}">
+            <dampingFactor>0.0005</dampingFactor>
+        </gazebo>
+        <link name="tibia_${suffix}">
+            <inertial>
+                <origin xyz="0 0 0" rpy="0 0 0"/>
+                <mass value="0.324357719"/>
+                <inertia ixx="0.0051411124" ixy="-0.00057530255" ixz="-0.000024729049" iyy="0.0081915737"
+                         iyz="-0.000019223094" izz="0.0011379812"/>
+            </inertial>
+            <visual>
+                <origin xyz="0 0 0" rpy="0 0 0"/>
+                <geometry>
+                    <mesh filename="package://phantomx_description/meshes/tibia_l.STL" scale="1 1 1"/>
+                </geometry>
+                <material name="Grey">
+                    <color rgba="0.20 0.20 0.20 1.0"/>
+                </material>
+            </visual>
+            <collision>
+                <origin xyz="0 0 0" rpy="0 0 0"/>
+                <geometry>
+                    <mesh filename="package://phantomx_description/meshes/tibia_l_coll.STL" scale="1 1 1"/>
+                </geometry>
+            </collision>
+        </link>
+        <gazebo reference="tibia_${suffix}">
+            <mu1>50.0</mu1>
+            <mu2>50.0</mu2>
+            <fdir1>0.000000 0.000000 0.000000</fdir1>
+            <kp>500000.0</kp>
+            <kd>10.0</kd>
+            <maxVel>0.00</maxVel>
+            <minDepth>0.001</minDepth>
+            <dampingFactor>0.0005</dampingFactor>
+            <selfCollide>1</selfCollide>
+        </gazebo>
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