Commit message: added real colours (#9)
* nom Alexndre

* add corentin

* Updated README.md with my name

* name

* added real colours

File: workspaceRos/src/phantomx/phantomx_description/urdf/phantomx_urdf.xacro (robot description, xacro)
@@ -22,7 +22,4 @@
                     <mesh filename="package://phantomx_description/meshes/body.STL" scale="1 1 1"/>
                 </geometry>
-                <material name="Grey">
-                    <color rgba="0.20 0.20 0.20 1.0"/>
-                </material>
             </visual>
             <collision>
@@ -34,5 +31,5 @@
         </link>
         <gazebo reference="MP_BODY">
-            <material>Gazebo/Grey</material>
+            <material>Gazebo/YellowGlow</material>
         </gazebo>
         <xacro:leg_l xyz="0.1248 -0.06164  0.001116" rpy="0 4.7123 0.7853981633974483" suffix="rf"/>
@@ -57,7 +54,4 @@
                     <mesh filename="package://phantomx_description/meshes/connect.STL" scale="1 1 1"/>
                 </geometry>
-                <material name="Grey">
-                    <color rgba="0.20 0.20 0.20 1.0"/>
-                </material>
             </visual>
             <collision>
@@ -84,7 +78,4 @@
                     <mesh filename="package://phantomx_description/meshes/connect.STL" scale="1 1 1"/>
                 </geometry>
-                <material name="Grey">
-                    <color rgba="0.20 0.20 0.20 1.0"/>
-                </material>
             </visual>
             <collision>
@@ -110,7 +101,4 @@
                     <mesh filename="package://phantomx_description/meshes/thigh_l.STL" scale="1 1 1"/>
                 </geometry>
-                <material name="Grey">
-                    <color rgba="0.20 0.20 0.20 1.0"/>
-                </material>
             </visual>
             <collision>
@@ -136,7 +124,4 @@
                     <mesh filename="package://phantomx_description/meshes/tibia_l.STL" scale="1 1 1"/>
                 </geometry>
-                <material name="Grey">
-                    <color rgba="0.20 0.20 0.20 1.0"/>
-                </material>
             </visual>
             <collision>
@@ -215,14 +200,14 @@
         </transmission>
         <gazebo reference="c1_${suffix}">
-            <material>Gazebo/Grey</material>
+            <material>Gazebo/RedGlow</material>
         </gazebo>
         <gazebo reference="c2_${suffix}">
-            <material>Gazebo/Grey</material>
+            <material>Gazebo/GreenGlow</material>
         </gazebo>
         <gazebo reference="thigh_${suffix}">
-            <material>Gazebo/Grey</material>
+            <material>Gazebo/TurquoiseGlow</material>
         </gazebo>
         <gazebo reference="tibia_${suffix}">
-            <material>Gazebo/Grey</material>
+        	<material>Gazebo/PurpleGlow</material>
         </gazebo>
     </xacro:macro>

Commit message: # Ceci est la combinaison de 5 commits. # Ceci est le premier message de validation :
# Ceci est la combinaison de 2 commits.
# Ceci est le premier message de validation :

# Ceci est la combinaison de 2 commits.
# Ceci est le premier message de validation :

# Ceci est la combinaison de 6 commits.
# Ceci est le premier message de validation :

# Ceci est la combinaison de 3 commits.
# Ceci est le premier message de validation :

# Ceci est la combinaison de 2 commits.
# Ceci est le premier message de validation :

# Ceci est la combinaison de 2 commits.
# Ceci est le premier message de validation :

AjoutLidar

# Ceci est le message de validation numéro 2 :

add pictures

# Ceci est le message de validation numéro 2 :

Conneries liées à mon IDE. Faudra que je le change un jour.

# Ceci est le message de validation numéro 2 :

creation du package projet

# Ceci est le message de validation numéro 3 :

AjoutLidar

# Ceci est le message de validation numéro 2 :

add corentin

# Ceci est le message de validation numéro 3 :

add phil name

# Ceci est le message de validation numéro 4 :

Updated README.md with my name

# Ceci est le message de validation numéro 5 :

name

# Ceci est le message de validation numéro 6 :

Changement Nom

# Ceci est le message de validation numéro 2 :

add phil name

# Ceci est le message de validation numéro 2 :

contenu modifié

# Ceci est le message de validation numéro 2 :

readme

# Ceci est le message de validation numéro 3 :

added real colours (#9)

* nom Alexndre

* add corentin

* Updated README.md with my name

* name

* added real colours

# Ceci est le message de validation numéro 4 :

reports (#10)

* contenu modifié

* Update README.md

* readme

* debriefs and goals

# Ceci est le message de validation numéro 5 :

AjoutLidar

File: workspaceRos/src/phantomx/phantomx_description/urdf/phantomx_urdf.xacro (robot description, xacro)
@@ -4,4 +4,7 @@
     <xacro:property name="thigh_offset_y" value="-0.0645"/>
     <xacro:property name="thigh_offset_z" value="-0.0145"/>
+    <xacro:property name="lenght_lidar" value="0.04" />
+    <xacro:property name="radius_lidar" value="0.03" />
+    <xacro:property name="mass_lidar" value="0.1" />
     <xacro:macro name="phantomx" params="parent *origin">
         <joint name="j_phantomx_attachment" type="fixed">
@@ -10,4 +13,5 @@
             <insert_block name="origin"/>
         </joint>
+<!-- ############# Link ####################### -->
         <link name="MP_BODY">
             <inertial>
@@ -143,4 +147,5 @@
             <selfCollide>1</selfCollide>
         </gazebo>
+<!-- ################## Joint #################### -->
         <joint name="j_c1_${suffix}" type="revolute">
             <parent link="MP_BODY"/>
@@ -169,4 +174,5 @@
             <limit effort="2.8" velocity="5.6548668" lower="-2.6179939" upper="2.6179939"/>
         </joint>
+<!-- ################### transmission ##################### -->
         <transmission name="t_c1_${suffix}">
             <type>transmission_interface/SimpleTransmission</type>
@@ -199,4 +205,5 @@
             </actuator>
         </transmission>
+<!-- ###################### reference #################### -->
         <gazebo reference="c1_${suffix}">
             <material>Gazebo/RedGlow</material>
@@ -212,3 +219,31 @@
         </gazebo>
     </xacro:macro>
+<!--  ###################  Lidar ###################### -->
+<link name="lidar">
+    <collision>
+        <geometry>
+            <cylinder length="${lenght_lidar}" radius="${radius_lidar}"/>
+            <origin rpy="0 0 0" xyz="0 0 ${-lenght_lidar/2}}"/>
+        </geometry>
+    </collision>
+    <visual>
+        <geometry>
+            <cylinder length="${lenght_lidar}" radius="${radius_lidar}"/>
+            <origin rpy="0 0 0" xyz="0 0 ${-lenght_lidar/2}"/>
+        </geometry>
+        <material name="red"/>
+    </visual>
+    <inertial>
+        <mass value="0"/>
+        <inertia
+            ixx="${mass_lidar*lenght_lidar*lenght_lidar/12.0+mass_lidar*radius_lidar*radius_lidar/2.0}" ixy="0.0" ixz="0.0"
+            iyy="${mass_lidar*lenght_lidar*lenght_lidar/12.0+mass_lidar*radius_lidar*radius_lidar/2.0}" iyz="0.0"
+            izz="${mass_lidar*radius_lidar*radius_lidar}"/>
+    </inertial>
+</link>
+<joint name="lidar_joint" type="fixed">
+    <parent link="MP_BODY"/>
+    <child link="lidar"/>
+    <origin rpy="0 0 0" xyz="0 0 ${0.045/2+lenght_lidar/2}"/>
+</joint>
 </robot>

Commit message: Camera update (#15)
* Update README.md

* readme

* debriefs and goals

* camera

* camera update

* camera update

* camera3d

Co-authored-by: ymusell <57345152+ymusell@users.noreply.github.com>
Co-authored-by: AlexandreCourjaud <38203726+AlexandreCourjaud@users.noreply.github.com>

File: workspaceRos/src/phantomx/phantomx_description/urdf/phantomx_urdf.xacro (robot description, xacro)
@@ -219,4 +219,5 @@
         </gazebo>
     </xacro:macro>
+<<<<<<< HEAD
 <!--  ###################  Lidar ###################### -->
 <link name="lidar">
@@ -247,3 +248,104 @@
     <origin rpy="0 0 0" xyz="0 0 ${0.045/2+lenght_lidar/2}"/>
 </joint>
+    <!-- ################################################################# -->
+    <!-- ###    Camera  ################################################## -->
+    <!-- ################################################################# -->
+    <!-- Add camera object -->
+    <link name="camera">
+        <visual>
+            <geometry>
+                <box size="0.02 0.02 0.02" />
+            </geometry>
+        </visual>
+    </link>
+    <!-- Add wonderful color to camera -->
+    <gazebo reference="camera">
+        <material>Gazebo/BlueGlow</material>
+    </gazebo>
+    <!-- Add link between camera and body object -->
+    <joint name="body2camera" type="fixed">
+        <parent link="MP_BODY"/>
+        <child link="camera"/>
+        <origin rpy="0 0 0" xyz="0.11 0 0"/>
+    </joint>
+    <!-- Add camera description
+    <gazebo reference="camera">
+        <sensor type="camera" name="camera1">
+            <update_rate>30.0</update_rate>
+            <camera name="head">
+                <horizontal_fov>1.3962634</horizontal_fov>
+                <image>
+                    <width>800</width>
+                    <height>800</height>
+                    <format>R8G8B8</format>
+                </image>
+                <clip>
+                    <near>0.02</near>
+                    <far>300</far>
+                </clip>
+                <noise>
+                    <type>gaussian</type>
+                    <mean>0.0</mean>
+                    <stddev>0.007</stddev>
+                </noise>
+            </camera>
+            <plugin name="camera_controller" filename="libgazebo_ros_camera.so">
+            <alwaysOn>true</alwaysOn>
+            <updateRate>0.0</updateRate>
+            <cameraName>rrbot/camera1</cameraName>
+            <imageTopicName>image_raw</imageTopicName>
+            <cameraInfoTopicName>camera_info</cameraInfoTopicName>
+            <frameName>camera_link</frameName>
+            <hackBaseline>0.07</hackBaseline>
+            <distortionK1>0.0</distortionK1>
+            <distortionK2>0.0</distortionK2>
+            <distortionK3>0.0</distortionK3>
+            <distortionT1>0.0</distortionT1>
+            <distortionT2>0.0</distortionT2>
+            </plugin>
+        </sensor>
+    </gazebo> -->
+    <gazebo reference="camera">
+        <sensor name='camera1' type='depth'>
+            <always_on>1</always_on>
+            <visualize>1</visualize>
+            <camera name='head'>
+                <horizontal_fov>1.047</horizontal_fov>
+                    <image>
+                    <width>640</width>
+                    <height>480</height>
+                    <format>R8G8B8</format>
+                </image>
+                <depth_camera>
+                    <output>depths</output>
+                </depth_camera>
+                <clip>
+                    <near>0.1</near>
+                    <far>100</far>
+                </clip>
+            </camera>
+            <plugin name='camera_controller' filename='libgazebo_ros_openni_kinect.so'>
+            <alwaysOn>true</alwaysOn>
+            <updateRate>30.0</updateRate>
+            <cameraName>camera</cameraName>
+            <frameName>/camera_link</frameName>
+            <imageTopicName>rgb/image_raw</imageTopicName>
+            <depthImageTopicName>depth/image_raw</depthImageTopicName>
+            <pointCloudTopicName>depth/points</pointCloudTopicName>
+            <cameraInfoTopicName>rgb/camera_info</cameraInfoTopicName>
+            <depthImageCameraInfoTopicName>depth/camera_info</depthImageCameraInfoTopicName>
+            <pointCloudCutoff>0.4</pointCloudCutoff>
+            <hackBaseline>0.07</hackBaseline>
+            <distortionK1>0.0</distortionK1>
+            <distortionK2>0.0</distortionK2>
+            <distortionK3>0.0</distortionK3>
+            <distortionT1>0.0</distortionT1>
+            <distortionT2>0.0</distortionT2>
+            <CxPrime>0.0</CxPrime>
+            <Cx>0.0</Cx>
+            <Cy>0.0</Cy>
+            <focalLength>0.0</focalLength>
+            </plugin>
+        </sensor>
+    </gazebo>
 </robot>

Commit message: conflict resolution

File: workspaceRos/src/phantomx/phantomx_description/urdf/phantomx_urdf.xacro (robot description, xacro)
@@ -391,4 +391,49 @@
         </sensor>
     </gazebo>
+<!--  ###################  Centrale inertielle ###################### -->
+<joint name="imu_joint" type="fixed">
+<axis xyz="1 0 0"/>
+<origin xyz="0 0 0.19"/>
+<parent link="MP_BODY"/>
+<child link="imu_link"/>
+</joint>
+<link name="imu_link">
+	<inertial>
+		<mass value="0.001"/>
+		<origin rpy="0 0 0" xyz="0 0 0"/>
+		<inertia ixx="0.0001" ixy="0" ixz="0" iyy="0.000001" iyz="0" izz="0.0001"/>
+	</inertial>
+	<visual>
+		<origin rpy="0 0 0" xyz="0 0 0"/>
+		<geometry>
+			<box size="0.001 0.001 0.001"/>
+		</geometry>
+	</visual>
+	<collision>
+		<origin rpy="0 0 0" xyz="0 0 0"/>
+		<geometry>
+			<box size=".001 .001 .001"/>
+		</geometry>
+	</collision>
+</link>
+<gazebo reference="imu_link">
+	<gravity>true</gravity>
+	<sensor name="imu_sensor" type="imu">
+		<always_on>true</always_on>
+		<update_rate>100</update_rate>
+		<visualize>true</visualize>
+		<topic>__default_topic__</topic>
+		<plugin filename="libgazebo_ros_imu_sensor.so" name="imu_plugin">
+			<topicName>phantomx/imu</topicName>
+			<bodyName>imu_link</bodyName>
+			<updateRateHZ>10.0</updateRateHZ>
+			<gaussianNoise>0.0</gaussianNoise>
+			<xyzOffset>0 0 0</xyzOffset>
+			<rpyOffset>0 0 0</rpyOffset>
+			<frameName>imu_link</frameName>
+		</plugin>
+		<pose>0 0 0 0 0 0</pose>
+	</sensor>
+</gazebo>
     <!--  ###################  Centrale inertielle ###################### -->
     <joint name="imu_joint" type="fixed">

Commit message: conflict resolution

File: workspaceRos/src/phantomx/phantomx_description/urdf/phantomx_urdf.xacro (robot description, xacro)
@@ -219,5 +219,4 @@
         </gazebo>
     </xacro:macro>
-<<<<<<< HEAD
 <!--  ###################  Lidar ###################### -->
 <link name="lidar">
@@ -349,3 +348,48 @@
         </sensor>
     </gazebo>
+<!--  ###################  Centrale inertielle ###################### -->
+<joint name="imu_joint" type="fixed">
+<axis xyz="1 0 0"/>
+<origin xyz="0 0 0.19"/>
+<parent link="MP_BODY"/>
+<child link="imu_link"/>
+</joint>
+<link name="imu_link">
+	<inertial>
+		<mass value="0.001"/>
+		<origin rpy="0 0 0" xyz="0 0 0"/>
+		<inertia ixx="0.0001" ixy="0" ixz="0" iyy="0.000001" iyz="0" izz="0.0001"/>
+	</inertial>
+	<visual>
+		<origin rpy="0 0 0" xyz="0 0 0"/>
+		<geometry>
+			<box size="0.001 0.001 0.001"/>
+		</geometry>
+	</visual>
+	<collision>
+		<origin rpy="0 0 0" xyz="0 0 0"/>
+		<geometry>
+			<box size=".001 .001 .001"/>
+		</geometry>
+	</collision>
+</link>
+<gazebo reference="imu_link">
+	<gravity>true</gravity>
+	<sensor name="imu_sensor" type="imu">
+		<always_on>true</always_on>
+		<update_rate>100</update_rate>
+		<visualize>true</visualize>
+		<topic>__default_topic__</topic>
+		<plugin filename="libgazebo_ros_imu_sensor.so" name="imu_plugin">
+			<topicName>phantomx/imu</topicName>
+			<bodyName>imu_link</bodyName>
+			<updateRateHZ>10.0</updateRateHZ>
+			<gaussianNoise>0.0</gaussianNoise>
+			<xyzOffset>0 0 0</xyzOffset>
+			<rpyOffset>0 0 0</rpyOffset>
+			<frameName>imu_link</frameName>
+		</plugin>
+		<pose>0 0 0 0 0 0</pose>
+	</sensor>
+</gazebo>
 </robot>

Commit message: IMU (#17)
* conflict resolution

*  la centrale inertielle // topic de publication /phantomx/imu

File: workspaceRos/src/phantomx/phantomx_description/urdf/phantomx_urdf.xacro (robot description, xacro)
@@ -348,3 +348,48 @@
         </sensor>
     </gazebo>
+<!--  ###################  Centrale inertielle ###################### -->
+<joint name="imu_joint" type="fixed">
+<axis xyz="1 0 0"/>
+<origin xyz="0 0 0.19"/>
+<parent link="MP_BODY"/>
+<child link="imu_link"/>
+</joint>
+<link name="imu_link">
+	<inertial>
+		<mass value="0.001"/>
+		<origin rpy="0 0 0" xyz="0 0 0"/>
+		<inertia ixx="0.0001" ixy="0" ixz="0" iyy="0.000001" iyz="0" izz="0.0001"/>
+	</inertial>
+	<visual>
+		<origin rpy="0 0 0" xyz="0 0 0"/>
+		<geometry>
+			<box size="0.001 0.001 0.001"/>
+		</geometry>
+	</visual>
+	<collision>
+		<origin rpy="0 0 0" xyz="0 0 0"/>
+		<geometry>
+			<box size=".001 .001 .001"/>
+		</geometry>
+	</collision>
+</link>
+<gazebo reference="imu_link">
+	<gravity>true</gravity>
+	<sensor name="imu_sensor" type="imu">
+		<always_on>true</always_on>
+		<update_rate>100</update_rate>
+		<visualize>true</visualize>
+		<topic>__default_topic__</topic>
+		<plugin filename="libgazebo_ros_imu_sensor.so" name="imu_plugin">
+			<topicName>phantomx/imu</topicName>
+			<bodyName>imu_link</bodyName>
+			<updateRateHZ>10.0</updateRateHZ>
+			<gaussianNoise>0.0</gaussianNoise>
+			<xyzOffset>0 0 0</xyzOffset>
+			<rpyOffset>0 0 0</rpyOffset>
+			<frameName>imu_link</frameName>
+		</plugin>
+		<pose>0 0 0 0 0 0</pose>
+	</sensor>
+</gazebo>
 </robot>

Commit message: camera 3d update and display (#20)
* Update README.md

* readme

* debriefs and goals

* camera

* camera update

* camera update

* Update README.md

* readme

* camera

* camera update

* visualization camera

* camera3d update

* camera3d update

* camera update

* visualization camera

* camera3d update

Co-authored-by: ymusell <57345152+ymusell@users.noreply.github.com>
Co-authored-by: AlexandreCourjaud <38203726+AlexandreCourjaud@users.noreply.github.com>

File: workspaceRos/src/phantomx/phantomx_description/urdf/phantomx_urdf.xacro (robot description, xacro)
@@ -299,41 +299,4 @@
         <origin rpy="0 0 0" xyz="0.11 0 0"/>
     </joint>
-    <!-- Add camera description
-    <gazebo reference="camera">
-        <sensor type="camera" name="camera1">
-            <update_rate>30.0</update_rate>
-            <camera name="head">
-                <horizontal_fov>1.3962634</horizontal_fov>
-                <image>
-                    <width>800</width>
-                    <height>800</height>
-                    <format>R8G8B8</format>
-                </image>
-                <clip>
-                    <near>0.02</near>
-                    <far>300</far>
-                </clip>
-                <noise>
-                    <type>gaussian</type>
-                    <mean>0.0</mean>
-                    <stddev>0.007</stddev>
-                </noise>
-            </camera>
-            <plugin name="camera_controller" filename="libgazebo_ros_camera.so">
-            <alwaysOn>true</alwaysOn>
-            <updateRate>0.0</updateRate>
-            <cameraName>rrbot/camera1</cameraName>
-            <imageTopicName>image_raw</imageTopicName>
-            <cameraInfoTopicName>camera_info</cameraInfoTopicName>
-            <frameName>camera_link</frameName>
-            <hackBaseline>0.07</hackBaseline>
-            <distortionK1>0.0</distortionK1>
-            <distortionK2>0.0</distortionK2>
-            <distortionK3>0.0</distortionK3>
-            <distortionT1>0.0</distortionT1>
-            <distortionT2>0.0</distortionT2>
-            </plugin>
-        </sensor>
-    </gazebo> -->
     <gazebo reference="camera">
         <sensor name='camera1' type='depth'>
@@ -355,7 +318,7 @@
                 </clip>
             </camera>
-            <plugin name='camera_controller' filename='libgazebo_ros_openni_kinect.so'>
+            <plugin name='camera_plugin' filename='libgazebo_ros_openni_kinect.so'>
             <alwaysOn>true</alwaysOn>
-            <updateRate>30.0</updateRate>
+            <updateRate>10.0</updateRate>
             <cameraName>camera</cameraName>
             <frameName>/camera_link</frameName>
@@ -366,4 +329,5 @@
             <depthImageCameraInfoTopicName>depth/camera_info</depthImageCameraInfoTopicName>
             <pointCloudCutoff>0.4</pointCloudCutoff>
+            <pointCloudCutoffMax>20.0</pointCloudCutoffMax>
             <hackBaseline>0.07</hackBaseline>
             <distortionK1>0.0</distortionK1>
@@ -379,48 +343,48 @@
         </sensor>
     </gazebo>
-<!--  ###################  Centrale inertielle ###################### -->
-<joint name="imu_joint" type="fixed">
-<axis xyz="1 0 0"/>
-<origin xyz="0 0 0.19"/>
-<parent link="MP_BODY"/>
-<child link="imu_link"/>
-</joint>
-<link name="imu_link">
-	<inertial>
-		<mass value="0.001"/>
-		<origin rpy="0 0 0" xyz="0 0 0"/>
-		<inertia ixx="0.0001" ixy="0" ixz="0" iyy="0.000001" iyz="0" izz="0.0001"/>
-	</inertial>
-	<visual>
-		<origin rpy="0 0 0" xyz="0 0 0"/>
-		<geometry>
-			<box size="0.001 0.001 0.001"/>
-		</geometry>
-	</visual>
-	<collision>
-		<origin rpy="0 0 0" xyz="0 0 0"/>
-		<geometry>
-			<box size=".001 .001 .001"/>
-		</geometry>
-	</collision>
-</link>
-<gazebo reference="imu_link">
-	<gravity>true</gravity>
-	<sensor name="imu_sensor" type="imu">
-		<always_on>true</always_on>
-		<update_rate>100</update_rate>
-		<visualize>true</visualize>
-		<topic>__default_topic__</topic>
-		<plugin filename="libgazebo_ros_imu_sensor.so" name="imu_plugin">
-			<topicName>phantomx/imu</topicName>
-			<bodyName>imu_link</bodyName>
-			<updateRateHZ>10.0</updateRateHZ>
-			<gaussianNoise>0.0</gaussianNoise>
-			<xyzOffset>0 0 0</xyzOffset>
-			<rpyOffset>0 0 0</rpyOffset>
-			<frameName>imu_link</frameName>
-		</plugin>
-		<pose>0 0 0 0 0 0</pose>
-	</sensor>
-</gazebo>
+    <!--  ###################  Centrale inertielle ###################### -->
+    <joint name="imu_joint" type="fixed">
+    <axis xyz="1 0 0"/>
+    <origin xyz="0 0 0.19"/>
+    <parent link="MP_BODY"/>
+    <child link="imu_link"/>
+    </joint>
+    <link name="imu_link">
+    	<inertial>
+    		<mass value="0.001"/>
+    		<origin rpy="0 0 0" xyz="0 0 0"/>
+    		<inertia ixx="0.0001" ixy="0" ixz="0" iyy="0.000001" iyz="0" izz="0.0001"/>
+    	</inertial>
+    	<visual>
+    		<origin rpy="0 0 0" xyz="0 0 0"/>
+    		<geometry>
+    			<box size="0.001 0.001 0.001"/>
+    		</geometry>
+    	</visual>
+    	<collision>
+    		<origin rpy="0 0 0" xyz="0 0 0"/>
+    		<geometry>
+    			<box size=".001 .001 .001"/>
+    		</geometry>
+    	</collision>
+    </link>
+    <gazebo reference="imu_link">
+    	<gravity>true</gravity>
+    	<sensor name="imu_sensor" type="imu">
+    		<always_on>true</always_on>
+    		<update_rate>100</update_rate>
+    		<visualize>true</visualize>
+    		<topic>__default_topic__</topic>
+    		<plugin filename="libgazebo_ros_imu_sensor.so" name="imu_plugin">
+    			<topicName>phantomx/imu</topicName>
+    			<bodyName>imu_link</bodyName>
+    			<updateRateHZ>10.0</updateRateHZ>
+    			<gaussianNoise>0.0</gaussianNoise>
+    			<xyzOffset>0 0 0</xyzOffset>
+    			<rpyOffset>0 0 0</rpyOffset>
+    			<frameName>imu_link</frameName>
+    		</plugin>
+    		<pose>0 0 0 0 0 0</pose>
+    	</sensor>
+    </gazebo>
 </robot>
