Commit message: add lidar color (#28)
* add lidar range fetch in python

* optimize algorithm, add color to lidar

File: workspaceRos/src/phantomx/phantomx_description/urdf/phantomx_urdf.xacro (robot description, xacro)
@@ -4,5 +4,5 @@
     <xacro:property name="thigh_offset_y" value="-0.0645"/>
     <xacro:property name="thigh_offset_z" value="-0.0145"/>
-    <xacro:property name="lenght_lidar" value="0.04" />
+    <xacro:property name="lenght_lidar" value="0.08" />
     <xacro:property name="radius_lidar" value="0.03" />
     <xacro:property name="mass_lidar" value="0.1" />
@@ -244,5 +244,4 @@
             <origin rpy="0 0 0" xyz="0 0 ${-lenght_lidar/2}"/>
         </geometry>
-        <material name="red"/>
     </visual>
     <inertial>
@@ -262,5 +261,5 @@
     <sensor type="ray" name="head_hokuyo_sensor">
       <pose> 0 0 0 0 0</pose>
-      <visualize>true</visualize>
+      <visualize>false</visualize>
       <update_rate>5</update_rate>
       <ray>
@@ -290,4 +289,8 @@
     </sensor>
   </gazebo>
+  <!-- Add wonderful color to lidar -->
+    <gazebo reference="lidar">
+        <material>Gazebo/WhiteGlow</material>
+    </gazebo>
     <!-- ################################################################# -->
     <!-- ###    Camera  ################################################## -->

Commit message: positionnement

File: workspaceRos/src/phantomx/phantomx_description/urdf/phantomx_urdf.xacro (robot description, xacro)
@@ -436,50 +436,4 @@
     	</sensor>
     </gazebo>
-=======
-<!--  ###################  Centrale inertielle ###################### -->
-<joint name="imu_joint" type="fixed">
-<axis xyz="1 0 0"/>
-<origin xyz="0 0 0.19"/>
-<parent link="MP_BODY"/>
-<child link="imu_link"/>
-</joint>
-<link name="imu_link">
-	<inertial>
-		<mass value="0.001"/>
-		<origin rpy="0 0 0" xyz="0 0 0"/>
-		<inertia ixx="0.0001" ixy="0" ixz="0" iyy="0.000001" iyz="0" izz="0.0001"/>
-	</inertial>
-	<visual>
-		<origin rpy="0 0 0" xyz="0 0 0"/>
-		<geometry>
-			<box size="0.001 0.001 0.001"/>
-		</geometry>
-	</visual>
-	<collision>
-		<origin rpy="0 0 0" xyz="0 0 0"/>
-		<geometry>
-			<box size=".001 .001 .001"/>
-		</geometry>
-	</collision>
-</link>
-<gazebo reference="imu_link">
-	<gravity>true</gravity>
-	<sensor name="imu_sensor" type="imu">
-		<always_on>true</always_on>
-		<update_rate>100</update_rate>
-		<visualize>true</visualize>
-		<topic>__default_topic__</topic>
-		<plugin filename="libgazebo_ros_imu_sensor.so" name="imu_plugin">
-			<topicName>phantomx/imu</topicName>
-			<bodyName>imu_link</bodyName>
-			<updateRateHZ>10.0</updateRateHZ>
-			<gaussianNoise>0.0</gaussianNoise>
-			<xyzOffset>0 0 0</xyzOffset>
-			<rpyOffset>0 0 0</rpyOffset>
-			<frameName>imu_link</frameName>
-		</plugin>
-		<pose>0 0 0 0 0 0</pose>
-	</sensor>
-</gazebo>
 <gazebo>
     <plugin name="p3d_base_controller" filename="libgazebo_ros_p3d.so">
@@ -494,4 +448,5 @@
     </plugin>
 </gazebo>
+<<<<<<< HEAD
 <gazebo>
     <plugin name="p3d_base_controller" filename="libgazebo_ros_p3d.so">
@@ -506,3 +461,5 @@
     </plugin>
 </gazebo>
+=======
+>>>>>>> positionnement
 </robot>

Commit message: positionnement

File: workspaceRos/src/phantomx/phantomx_description/urdf/phantomx_urdf.xacro (robot description, xacro)
@@ -391,49 +391,49 @@
         </sensor>
     </gazebo>
-<!--  ###################  Centrale inertielle ###################### -->
-<joint name="imu_joint" type="fixed">
-<axis xyz="1 0 0"/>
-<origin xyz="0 0 0.19"/>
-<parent link="MP_BODY"/>
-<child link="imu_link"/>
-</joint>
-<link name="imu_link">
-	<inertial>
-		<mass value="0.001"/>
-		<origin rpy="0 0 0" xyz="0 0 0"/>
-		<inertia ixx="0.0001" ixy="0" ixz="0" iyy="0.000001" iyz="0" izz="0.0001"/>
-	</inertial>
-	<visual>
-		<origin rpy="0 0 0" xyz="0 0 0"/>
-		<geometry>
-			<box size="0.001 0.001 0.001"/>
-		</geometry>
-	</visual>
-	<collision>
-		<origin rpy="0 0 0" xyz="0 0 0"/>
-		<geometry>
-			<box size=".001 .001 .001"/>
-		</geometry>
-	</collision>
-</link>
-<gazebo reference="imu_link">
-	<gravity>true</gravity>
-	<sensor name="imu_sensor" type="imu">
-		<always_on>true</always_on>
-		<update_rate>100</update_rate>
-		<visualize>true</visualize>
-		<topic>__default_topic__</topic>
-		<plugin filename="libgazebo_ros_imu_sensor.so" name="imu_plugin">
-			<topicName>phantomx/imu</topicName>
-			<bodyName>imu_link</bodyName>
-			<updateRateHZ>10.0</updateRateHZ>
-			<gaussianNoise>0.0</gaussianNoise>
-			<xyzOffset>0 0 0</xyzOffset>
-			<rpyOffset>0 0 0</rpyOffset>
-			<frameName>imu_link</frameName>
-		</plugin>
-		<pose>0 0 0 0 0 0</pose>
-	</sensor>
-</gazebo>
+    <!--  ###################  Centrale inertielle ###################### -->
+    <joint name="imu_joint" type="fixed">
+    <axis xyz="1 0 0"/>
+    <origin xyz="0 0 0.19"/>
+    <parent link="MP_BODY"/>
+    <child link="imu_link"/>
+    </joint>
+    <link name="imu_link">
+    	<inertial>
+    		<mass value="0.001"/>
+    		<origin rpy="0 0 0" xyz="0 0 0"/>
+    		<inertia ixx="0.0001" ixy="0" ixz="0" iyy="0.000001" iyz="0" izz="0.0001"/>
+    	</inertial>
+    	<visual>
+    		<origin rpy="0 0 0" xyz="0 0 0"/>
+    		<geometry>
+    			<box size="0.001 0.001 0.001"/>
+    		</geometry>
+    	</visual>
+    	<collision>
+    		<origin rpy="0 0 0" xyz="0 0 0"/>
+    		<geometry>
+    			<box size=".001 .001 .001"/>
+    		</geometry>
+    	</collision>
+    </link>
+    <gazebo reference="imu_link">
+    	<gravity>true</gravity>
+    	<sensor name="imu_sensor" type="imu">
+    		<always_on>true</always_on>
+    		<update_rate>100</update_rate>
+    		<visualize>true</visualize>
+    		<topic>__default_topic__</topic>
+    		<plugin filename="libgazebo_ros_imu_sensor.so" name="imu_plugin">
+    			<topicName>phantomx/imu</topicName>
+    			<bodyName>imu_link</bodyName>
+    			<updateRateHZ>10.0</updateRateHZ>
+    			<gaussianNoise>0.0</gaussianNoise>
+    			<xyzOffset>0 0 0</xyzOffset>
+    			<rpyOffset>0 0 0</rpyOffset>
+    			<frameName>imu_link</frameName>
+    		</plugin>
+    		<pose>0 0 0 0 0 0</pose>
+    	</sensor>
+    </gazebo>
 <gazebo>
     <plugin name="p3d_base_controller" filename="libgazebo_ros_p3d.so">
@@ -448,6 +448,3 @@
     </plugin>
 </gazebo>
-<<<<<<< HEAD
-=======
->>>>>>> positionnement
 </robot>

Commit message: positionnement

File: workspaceRos/src/phantomx/phantomx_description/urdf/phantomx_urdf.xacro (robot description, xacro)
@@ -436,73 +436,4 @@
 	</sensor>
 </gazebo>
-    <!--  ###################  Centrale inertielle ###################### -->
-    <joint name="imu_joint" type="fixed">
-    <axis xyz="1 0 0"/>
-    <origin xyz="0 0 0.19"/>
-    <parent link="MP_BODY"/>
-    <child link="imu_link"/>
-    </joint>
-    <link name="imu_link">
-    	<inertial>
-    		<mass value="0.001"/>
-    		<origin rpy="0 0 0" xyz="0 0 0"/>
-    		<inertia ixx="0.0001" ixy="0" ixz="0" iyy="0.000001" iyz="0" izz="0.0001"/>
-    	</inertial>
-    	<visual>
-    		<origin rpy="0 0 0" xyz="0 0 0"/>
-    		<geometry>
-    			<box size="0.001 0.001 0.001"/>
-    		</geometry>
-    	</visual>
-    	<collision>
-    		<origin rpy="0 0 0" xyz="0 0 0"/>
-    		<geometry>
-    			<box size=".001 .001 .001"/>
-    		</geometry>
-    	</collision>
-    </link>
-    <gazebo reference="imu_link">
-    	<gravity>true</gravity>
-    	<sensor name="imu_sensor" type="imu">
-    		<always_on>true</always_on>
-    		<update_rate>100</update_rate>
-    		<visualize>true</visualize>
-    		<topic>__default_topic__</topic>
-    		<plugin filename="libgazebo_ros_imu_sensor.so" name="imu_plugin">
-    			<topicName>phantomx/imu</topicName>
-    			<bodyName>imu_link</bodyName>
-    			<updateRateHZ>10.0</updateRateHZ>
-    			<gaussianNoise>0.0</gaussianNoise>
-    			<xyzOffset>0 0 0</xyzOffset>
-    			<rpyOffset>0 0 0</rpyOffset>
-    			<frameName>imu_link</frameName>
-    		</plugin>
-    		<pose>0 0 0 0 0 0</pose>
-    	</sensor>
-    </gazebo>
-<gazebo>
-    <plugin name="p3d_base_controller" filename="libgazebo_ros_p3d.so">
-      <alwaysOn>true</alwaysOn>
-      <updateRate>50.0</updateRate>
-      <bodyName>MP_BODY</bodyName>
-      <topicName>ground_truth/state</topicName>
-      <gaussianNoise>0.01</gaussianNoise>
-      <frameName>world</frameName>
-      <xyzOffsets>0 0 0</xyzOffsets>
-      <rpyOffsets>0 0 0</rpyOffsets>
-    </plugin>
-</gazebo>
-<gazebo>
-    <plugin name="p3d_base_controller" filename="libgazebo_ros_p3d.so">
-      <alwaysOn>true</alwaysOn>
-      <updateRate>50.0</updateRate>
-      <bodyName>MP_BODY</bodyName>
-      <topicName>ground_truth/state</topicName>
-      <gaussianNoise>0.01</gaussianNoise>
-      <frameName>world</frameName>
-      <xyzOffsets>0 0 0</xyzOffsets>
-      <rpyOffsets>0 0 0</rpyOffsets>
-    </plugin>
-</gazebo>
 <gazebo>
     <plugin name="p3d_base_controller" filename="libgazebo_ros_p3d.so">

Commit message: positionnement

File: workspaceRos/src/phantomx/phantomx_description/urdf/phantomx_urdf.xacro (robot description, xacro)
@@ -436,62 +436,4 @@
     	</sensor>
     </gazebo>
-=======
-<!--  ###################  Centrale inertielle ###################### -->
-<joint name="imu_joint" type="fixed">
-<axis xyz="1 0 0"/>
-<origin xyz="0 0 0.19"/>
-<parent link="MP_BODY"/>
-<child link="imu_link"/>
-</joint>
-<link name="imu_link">
-	<inertial>
-		<mass value="0.001"/>
-		<origin rpy="0 0 0" xyz="0 0 0"/>
-		<inertia ixx="0.0001" ixy="0" ixz="0" iyy="0.000001" iyz="0" izz="0.0001"/>
-	</inertial>
-	<visual>
-		<origin rpy="0 0 0" xyz="0 0 0"/>
-		<geometry>
-			<box size="0.001 0.001 0.001"/>
-		</geometry>
-	</visual>
-	<collision>
-		<origin rpy="0 0 0" xyz="0 0 0"/>
-		<geometry>
-			<box size=".001 .001 .001"/>
-		</geometry>
-	</collision>
-</link>
-<gazebo reference="imu_link">
-	<gravity>true</gravity>
-	<sensor name="imu_sensor" type="imu">
-		<always_on>true</always_on>
-		<update_rate>100</update_rate>
-		<visualize>true</visualize>
-		<topic>__default_topic__</topic>
-		<plugin filename="libgazebo_ros_imu_sensor.so" name="imu_plugin">
-			<topicName>phantomx/imu</topicName>
-			<bodyName>imu_link</bodyName>
-			<updateRateHZ>10.0</updateRateHZ>
-			<gaussianNoise>0.0</gaussianNoise>
-			<xyzOffset>0 0 0</xyzOffset>
-			<rpyOffset>0 0 0</rpyOffset>
-			<frameName>imu_link</frameName>
-		</plugin>
-		<pose>0 0 0 0 0 0</pose>
-	</sensor>
-</gazebo>
-<gazebo>
-    <plugin name="p3d_base_controller" filename="libgazebo_ros_p3d.so">
-      <alwaysOn>true</alwaysOn>
-      <updateRate>50.0</updateRate>
-      <bodyName>MP_BODY</bodyName>
-      <topicName>ground_truth/state</topicName>
-      <gaussianNoise>0.01</gaussianNoise>
-      <frameName>world</frameName>
-      <xyzOffsets>0 0 0</xyzOffsets>
-      <rpyOffsets>0 0 0</rpyOffsets>
-    </plugin>
-</gazebo>
 <gazebo>
     <plugin name="p3d_base_controller" filename="libgazebo_ros_p3d.so">

Commit message: positionnement

File: workspaceRos/src/phantomx/phantomx_description/urdf/phantomx_urdf.xacro (robot description, xacro)
@@ -436,49 +436,4 @@
 	</sensor>
 </gazebo>
-    <!--  ###################  Centrale inertielle ###################### -->
-    <joint name="imu_joint" type="fixed">
-    <axis xyz="1 0 0"/>
-    <origin xyz="0 0 0.19"/>
-    <parent link="MP_BODY"/>
-    <child link="imu_link"/>
-    </joint>
-    <link name="imu_link">
-    	<inertial>
-    		<mass value="0.001"/>
-    		<origin rpy="0 0 0" xyz="0 0 0"/>
-    		<inertia ixx="0.0001" ixy="0" ixz="0" iyy="0.000001" iyz="0" izz="0.0001"/>
-    	</inertial>
-    	<visual>
-    		<origin rpy="0 0 0" xyz="0 0 0"/>
-    		<geometry>
-    			<box size="0.001 0.001 0.001"/>
-    		</geometry>
-    	</visual>
-    	<collision>
-    		<origin rpy="0 0 0" xyz="0 0 0"/>
-    		<geometry>
-    			<box size=".001 .001 .001"/>
-    		</geometry>
-    	</collision>
-    </link>
-    <gazebo reference="imu_link">
-    	<gravity>true</gravity>
-    	<sensor name="imu_sensor" type="imu">
-    		<always_on>true</always_on>
-    		<update_rate>100</update_rate>
-    		<visualize>true</visualize>
-    		<topic>__default_topic__</topic>
-    		<plugin filename="libgazebo_ros_imu_sensor.so" name="imu_plugin">
-    			<topicName>phantomx/imu</topicName>
-    			<bodyName>imu_link</bodyName>
-    			<updateRateHZ>10.0</updateRateHZ>
-    			<gaussianNoise>0.0</gaussianNoise>
-    			<xyzOffset>0 0 0</xyzOffset>
-    			<rpyOffset>0 0 0</rpyOffset>
-    			<frameName>imu_link</frameName>
-    		</plugin>
-    		<pose>0 0 0 0 0 0</pose>
-    	</sensor>
-    </gazebo>
 <gazebo>
     <plugin name="p3d_base_controller" filename="libgazebo_ros_p3d.so">
@@ -493,3 +448,6 @@
     </plugin>
 </gazebo>
+<<<<<<< HEAD
+=======
+>>>>>>> positionnement
 </robot>

Commit message: positionnement

File: workspaceRos/src/phantomx/phantomx_description/urdf/phantomx_urdf.xacro (robot description, xacro)
@@ -436,50 +436,4 @@
     	</sensor>
     </gazebo>
-=======
-<!--  ###################  Centrale inertielle ###################### -->
-<joint name="imu_joint" type="fixed">
-<axis xyz="1 0 0"/>
-<origin xyz="0 0 0.19"/>
-<parent link="MP_BODY"/>
-<child link="imu_link"/>
-</joint>
-<link name="imu_link">
-	<inertial>
-		<mass value="0.001"/>
-		<origin rpy="0 0 0" xyz="0 0 0"/>
-		<inertia ixx="0.0001" ixy="0" ixz="0" iyy="0.000001" iyz="0" izz="0.0001"/>
-	</inertial>
-	<visual>
-		<origin rpy="0 0 0" xyz="0 0 0"/>
-		<geometry>
-			<box size="0.001 0.001 0.001"/>
-		</geometry>
-	</visual>
-	<collision>
-		<origin rpy="0 0 0" xyz="0 0 0"/>
-		<geometry>
-			<box size=".001 .001 .001"/>
-		</geometry>
-	</collision>
-</link>
-<gazebo reference="imu_link">
-	<gravity>true</gravity>
-	<sensor name="imu_sensor" type="imu">
-		<always_on>true</always_on>
-		<update_rate>100</update_rate>
-		<visualize>true</visualize>
-		<topic>__default_topic__</topic>
-		<plugin filename="libgazebo_ros_imu_sensor.so" name="imu_plugin">
-			<topicName>phantomx/imu</topicName>
-			<bodyName>imu_link</bodyName>
-			<updateRateHZ>10.0</updateRateHZ>
-			<gaussianNoise>0.0</gaussianNoise>
-			<xyzOffset>0 0 0</xyzOffset>
-			<rpyOffset>0 0 0</rpyOffset>
-			<frameName>imu_link</frameName>
-		</plugin>
-		<pose>0 0 0 0 0 0</pose>
-	</sensor>
-</gazebo>
 <gazebo>
     <plugin name="p3d_base_controller" filename="libgazebo_ros_p3d.so">

Commit message: positionnement

File: workspaceRos/src/phantomx/phantomx_description/urdf/phantomx_urdf.xacro (robot description, xacro)
@@ -436,49 +436,4 @@
 	</sensor>
 </gazebo>
-    <!--  ###################  Centrale inertielle ###################### -->
-    <joint name="imu_joint" type="fixed">
-    <axis xyz="1 0 0"/>
-    <origin xyz="0 0 0.19"/>
-    <parent link="MP_BODY"/>
-    <child link="imu_link"/>
-    </joint>
-    <link name="imu_link">
-    	<inertial>
-    		<mass value="0.001"/>
-    		<origin rpy="0 0 0" xyz="0 0 0"/>
-    		<inertia ixx="0.0001" ixy="0" ixz="0" iyy="0.000001" iyz="0" izz="0.0001"/>
-    	</inertial>
-    	<visual>
-    		<origin rpy="0 0 0" xyz="0 0 0"/>
-    		<geometry>
-    			<box size="0.001 0.001 0.001"/>
-    		</geometry>
-    	</visual>
-    	<collision>
-    		<origin rpy="0 0 0" xyz="0 0 0"/>
-    		<geometry>
-    			<box size=".001 .001 .001"/>
-    		</geometry>
-    	</collision>
-    </link>
-    <gazebo reference="imu_link">
-    	<gravity>true</gravity>
-    	<sensor name="imu_sensor" type="imu">
-    		<always_on>true</always_on>
-    		<update_rate>100</update_rate>
-    		<visualize>true</visualize>
-    		<topic>__default_topic__</topic>
-    		<plugin filename="libgazebo_ros_imu_sensor.so" name="imu_plugin">
-    			<topicName>phantomx/imu</topicName>
-    			<bodyName>imu_link</bodyName>
-    			<updateRateHZ>10.0</updateRateHZ>
-    			<gaussianNoise>0.0</gaussianNoise>
-    			<xyzOffset>0 0 0</xyzOffset>
-    			<rpyOffset>0 0 0</rpyOffset>
-    			<frameName>imu_link</frameName>
-    		</plugin>
-    		<pose>0 0 0 0 0 0</pose>
-    	</sensor>
-    </gazebo>
 <gazebo>
     <plugin name="p3d_base_controller" filename="libgazebo_ros_p3d.so">

Commit message: positionnement

File: workspaceRos/src/phantomx/phantomx_description/urdf/phantomx_urdf.xacro (robot description, xacro)
@@ -391,49 +391,49 @@
         </sensor>
     </gazebo>
-<!--  ###################  Centrale inertielle ###################### -->
-<joint name="imu_joint" type="fixed">
-<axis xyz="1 0 0"/>
-<origin xyz="0 0 0.19"/>
-<parent link="MP_BODY"/>
-<child link="imu_link"/>
-</joint>
-<link name="imu_link">
-	<inertial>
-		<mass value="0.001"/>
-		<origin rpy="0 0 0" xyz="0 0 0"/>
-		<inertia ixx="0.0001" ixy="0" ixz="0" iyy="0.000001" iyz="0" izz="0.0001"/>
-	</inertial>
-	<visual>
-		<origin rpy="0 0 0" xyz="0 0 0"/>
-		<geometry>
-			<box size="0.001 0.001 0.001"/>
-		</geometry>
-	</visual>
-	<collision>
-		<origin rpy="0 0 0" xyz="0 0 0"/>
-		<geometry>
-			<box size=".001 .001 .001"/>
-		</geometry>
-	</collision>
-</link>
-<gazebo reference="imu_link">
-	<gravity>true</gravity>
-	<sensor name="imu_sensor" type="imu">
-		<always_on>true</always_on>
-		<update_rate>100</update_rate>
-		<visualize>true</visualize>
-		<topic>__default_topic__</topic>
-		<plugin filename="libgazebo_ros_imu_sensor.so" name="imu_plugin">
-			<topicName>phantomx/imu</topicName>
-			<bodyName>imu_link</bodyName>
-			<updateRateHZ>10.0</updateRateHZ>
-			<gaussianNoise>0.0</gaussianNoise>
-			<xyzOffset>0 0 0</xyzOffset>
-			<rpyOffset>0 0 0</rpyOffset>
-			<frameName>imu_link</frameName>
-		</plugin>
-		<pose>0 0 0 0 0 0</pose>
-	</sensor>
-</gazebo>
+    <!--  ###################  Centrale inertielle ###################### -->
+    <joint name="imu_joint" type="fixed">
+    <axis xyz="1 0 0"/>
+    <origin xyz="0 0 0.19"/>
+    <parent link="MP_BODY"/>
+    <child link="imu_link"/>
+    </joint>
+    <link name="imu_link">
+    	<inertial>
+    		<mass value="0.001"/>
+    		<origin rpy="0 0 0" xyz="0 0 0"/>
+    		<inertia ixx="0.0001" ixy="0" ixz="0" iyy="0.000001" iyz="0" izz="0.0001"/>
+    	</inertial>
+    	<visual>
+    		<origin rpy="0 0 0" xyz="0 0 0"/>
+    		<geometry>
+    			<box size="0.001 0.001 0.001"/>
+    		</geometry>
+    	</visual>
+    	<collision>
+    		<origin rpy="0 0 0" xyz="0 0 0"/>
+    		<geometry>
+    			<box size=".001 .001 .001"/>
+    		</geometry>
+    	</collision>
+    </link>
+    <gazebo reference="imu_link">
+    	<gravity>true</gravity>
+    	<sensor name="imu_sensor" type="imu">
+    		<always_on>true</always_on>
+    		<update_rate>100</update_rate>
+    		<visualize>true</visualize>
+    		<topic>__default_topic__</topic>
+    		<plugin filename="libgazebo_ros_imu_sensor.so" name="imu_plugin">
+    			<topicName>phantomx/imu</topicName>
+    			<bodyName>imu_link</bodyName>
+    			<updateRateHZ>10.0</updateRateHZ>
+    			<gaussianNoise>0.0</gaussianNoise>
+    			<xyzOffset>0 0 0</xyzOffset>
+    			<rpyOffset>0 0 0</rpyOffset>
+    			<frameName>imu_link</frameName>
+    		</plugin>
+    		<pose>0 0 0 0 0 0</pose>
+    	</sensor>
+    </gazebo>
 <gazebo>
     <plugin name="p3d_base_controller" filename="libgazebo_ros_p3d.so">

Commit message: mod 4

File: workspaceRos/src/phantomx/phantomx_description/urdf/phantomx_urdf.xacro (robot description, xacro)
@@ -436,4 +436,62 @@
     	</sensor>
     </gazebo>
+=======
+<!--  ###################  Centrale inertielle ###################### -->
+<joint name="imu_joint" type="fixed">
+<axis xyz="1 0 0"/>
+<origin xyz="0 0 0.19"/>
+<parent link="MP_BODY"/>
+<child link="imu_link"/>
+</joint>
+<link name="imu_link">
+	<inertial>
+		<mass value="0.001"/>
+		<origin rpy="0 0 0" xyz="0 0 0"/>
+		<inertia ixx="0.0001" ixy="0" ixz="0" iyy="0.000001" iyz="0" izz="0.0001"/>
+	</inertial>
+	<visual>
+		<origin rpy="0 0 0" xyz="0 0 0"/>
+		<geometry>
+			<box size="0.001 0.001 0.001"/>
+		</geometry>
+	</visual>
+	<collision>
+		<origin rpy="0 0 0" xyz="0 0 0"/>
+		<geometry>
+			<box size=".001 .001 .001"/>
+		</geometry>
+	</collision>
+</link>
+<gazebo reference="imu_link">
+	<gravity>true</gravity>
+	<sensor name="imu_sensor" type="imu">
+		<always_on>true</always_on>
+		<update_rate>100</update_rate>
+		<visualize>true</visualize>
+		<topic>__default_topic__</topic>
+		<plugin filename="libgazebo_ros_imu_sensor.so" name="imu_plugin">
+			<topicName>phantomx/imu</topicName>
+			<bodyName>imu_link</bodyName>
+			<updateRateHZ>10.0</updateRateHZ>
+			<gaussianNoise>0.0</gaussianNoise>
+			<xyzOffset>0 0 0</xyzOffset>
+			<rpyOffset>0 0 0</rpyOffset>
+			<frameName>imu_link</frameName>
+		</plugin>
+		<pose>0 0 0 0 0 0</pose>
+	</sensor>
+</gazebo>
+<gazebo>
+    <plugin name="p3d_base_controller" filename="libgazebo_ros_p3d.so">
+      <alwaysOn>true</alwaysOn>
+      <updateRate>50.0</updateRate>
+      <bodyName>MP_BODY</bodyName>
+      <topicName>ground_truth/state</topicName>
+      <gaussianNoise>0.01</gaussianNoise>
+      <frameName>world</frameName>
+      <xyzOffsets>0 0 0</xyzOffsets>
+      <rpyOffsets>0 0 0</rpyOffsets>
+    </plugin>
+</gazebo>
 <gazebo>
     <plugin name="p3d_base_controller" filename="libgazebo_ros_p3d.so">
