Commit message: add goal 3 (#34)
* add lidar range fetch in python

* optimize algorithm, add color to lidar

* add goal3

* update goal3

File: workspaceRos/src/phantomx/phantomx_description/urdf/phantomx_urdf.xacro (robot description, xacro)
@@ -391,30 +391,30 @@
         </sensor>
     </gazebo>
-    <!--  ###################  Centrale inertielle ###################### -->
-    <joint name="imu_joint" type="fixed">
-    <axis xyz="1 0 0"/>
-    <origin xyz="0 0 0.19"/>
-    <parent link="MP_BODY"/>
-    <child link="imu_link"/>
-    </joint>
-    <link name="imu_link">
-    	<inertial>
-    		<mass value="0.001"/>
-    		<origin rpy="0 0 0" xyz="0 0 0"/>
-    		<inertia ixx="0.0001" ixy="0" ixz="0" iyy="0.000001" iyz="0" izz="0.0001"/>
-    	</inertial>
-    	<visual>
-    		<origin rpy="0 0 0" xyz="0 0 0"/>
-    		<geometry>
-    			<box size="0.001 0.001 0.001"/>
-    		</geometry>
-    	</visual>
-    	<collision>
-    		<origin rpy="0 0 0" xyz="0 0 0"/>
-    		<geometry>
-    			<box size=".001 .001 .001"/>
-    		</geometry>
-    	</collision>
-    </link>
+<!--  ###################  Centrale inertielle ###################### -->
+<joint name="imu_joint" type="fixed">
+<axis xyz="1 0 0"/>
+<origin xyz="0 0 0.19"/>
+<parent link="MP_BODY"/>
+<child link="imu_link"/>
+</joint>
+<link name="imu_link">
+	<inertial>
+		<mass value="0.001"/>
+		<origin rpy="0 0 0" xyz="0 0 0"/>
+		<inertia ixx="0.0001" ixy="0" ixz="0" iyy="0.000001" iyz="0" izz="0.0001"/>
+	</inertial>
+	<visual>
+		<origin rpy="0 0 0" xyz="0 0 0"/>
+		<geometry>
+			<box size="0.001 0.001 0.001"/>
+		</geometry>
+	</visual>
+	<collision>
+		<origin rpy="0 0 0" xyz="0 0 0"/>
+		<geometry>
+			<box size=".001 .001 .001"/>
+		</geometry>
+	</collision>
+</link>
 <gazebo reference="imu_link">
 	<gravity>true</gravity>
@@ -448,15 +448,3 @@
     </plugin>
 </gazebo>
-<gazebo>
-    <plugin name="p3d_base_controller" filename="libgazebo_ros_p3d.so">
-      <alwaysOn>true</alwaysOn>
-      <updateRate>50.0</updateRate>
-      <bodyName>MP_BODY</bodyName>
-      <topicName>ground_truth/state</topicName>
-      <gaussianNoise>0.01</gaussianNoise>
-      <frameName>world</frameName>
-      <xyzOffsets>0 0 0</xyzOffsets>
-      <rpyOffsets>0 0 0</rpyOffsets>
-    </plugin>
-</gazebo>
 </robot>

Commit message: add goal 3 (#34)
* add lidar range fetch in python

* optimize algorithm, add color to lidar

* add goal3

* update goal3

File: workspaceRos/src/phantomx/phantomx_description/urdf/phantomx_urdf.xacro (robot description, xacro)
@@ -391,30 +391,30 @@
         </sensor>
     </gazebo>
-    <!--  ###################  Centrale inertielle ###################### -->
-    <joint name="imu_joint" type="fixed">
-    <axis xyz="1 0 0"/>
-    <origin xyz="0 0 0.19"/>
-    <parent link="MP_BODY"/>
-    <child link="imu_link"/>
-    </joint>
-    <link name="imu_link">
-    	<inertial>
-    		<mass value="0.001"/>
-    		<origin rpy="0 0 0" xyz="0 0 0"/>
-    		<inertia ixx="0.0001" ixy="0" ixz="0" iyy="0.000001" iyz="0" izz="0.0001"/>
-    	</inertial>
-    	<visual>
-    		<origin rpy="0 0 0" xyz="0 0 0"/>
-    		<geometry>
-    			<box size="0.001 0.001 0.001"/>
-    		</geometry>
-    	</visual>
-    	<collision>
-    		<origin rpy="0 0 0" xyz="0 0 0"/>
-    		<geometry>
-    			<box size=".001 .001 .001"/>
-    		</geometry>
-    	</collision>
-    </link>
+<!--  ###################  Centrale inertielle ###################### -->
+<joint name="imu_joint" type="fixed">
+<axis xyz="1 0 0"/>
+<origin xyz="0 0 0.19"/>
+<parent link="MP_BODY"/>
+<child link="imu_link"/>
+</joint>
+<link name="imu_link">
+	<inertial>
+		<mass value="0.001"/>
+		<origin rpy="0 0 0" xyz="0 0 0"/>
+		<inertia ixx="0.0001" ixy="0" ixz="0" iyy="0.000001" iyz="0" izz="0.0001"/>
+	</inertial>
+	<visual>
+		<origin rpy="0 0 0" xyz="0 0 0"/>
+		<geometry>
+			<box size="0.001 0.001 0.001"/>
+		</geometry>
+	</visual>
+	<collision>
+		<origin rpy="0 0 0" xyz="0 0 0"/>
+		<geometry>
+			<box size=".001 .001 .001"/>
+		</geometry>
+	</collision>
+</link>
 <gazebo reference="imu_link">
 	<gravity>true</gravity>

Commit message: modification final du sprint

File: workspaceRos/src/phantomx/phantomx_description/urdf/phantomx_urdf.xacro (robot description, xacro)
@@ -391,52 +391,4 @@
         </sensor>
     </gazebo>
-<<<<<<< HEAD
-<!--  ###################  Centrale inertielle ###################### -->
-<joint name="imu_joint" type="fixed">
-<axis xyz="1 0 0"/>
-<origin xyz="0 0 0.19"/>
-<parent link="MP_BODY"/>
-<child link="imu_link"/>
-</joint>
-<link name="imu_link">
-	<inertial>
-		<mass value="0.001"/>
-		<origin rpy="0 0 0" xyz="0 0 0"/>
-		<inertia ixx="0.0001" ixy="0" ixz="0" iyy="0.000001" iyz="0" izz="0.0001"/>
-	</inertial>
-	<visual>
-		<origin rpy="0 0 0" xyz="0 0 0"/>
-		<geometry>
-			<box size="0.001 0.001 0.001"/>
-		</geometry>
-	</visual>
-	<collision>
-		<origin rpy="0 0 0" xyz="0 0 0"/>
-		<geometry>
-			<box size=".001 .001 .001"/>
-		</geometry>
-	</collision>
-</link>
-<gazebo reference="imu_link">
-	<gravity>true</gravity>
-	<sensor name="imu_sensor" type="imu">
-		<always_on>true</always_on>
-		<update_rate>100</update_rate>
-		<visualize>true</visualize>
-		<topic>__default_topic__</topic>
-		<plugin filename="libgazebo_ros_imu_sensor.so" name="imu_plugin">
-			<topicName>phantomx/imu</topicName>
-			<bodyName>imu_link</bodyName>
-			<updateRateHZ>10.0</updateRateHZ>
-			<gaussianNoise>0.0</gaussianNoise>
-			<xyzOffset>0 0 0</xyzOffset>
-			<rpyOffset>0 0 0</rpyOffset>
-			<frameName>imu_link</frameName>
-		</plugin>
-		<pose>0 0 0 0 0 0</pose>
-	</sensor>
-</gazebo>
-=======
->>>>>>> positionnement
     <!--  ###################  Centrale inertielle ###################### -->
     <joint name="imu_joint" type="fixed">
@@ -484,7 +436,4 @@
     	</sensor>
     </gazebo>
-<<<<<<< HEAD
-=======
->>>>>>> positionnement
 <gazebo>
     <plugin name="p3d_base_controller" filename="libgazebo_ros_p3d.so">
@@ -499,6 +448,3 @@
     </plugin>
 </gazebo>
-<<<<<<< HEAD
-=======
->>>>>>> positionnement
 </robot>
